Commit message: added landing platform

File: rotors_description/urdf/hummingbird.xacro (robot description, xacro)
@@ -37,4 +37,5 @@
   <xacro:property name="rotor_drag_coefficient" value="8.06428e-05" />
   <xacro:property name="rolling_moment_coefficient" value="0.000001" />
+  <xacro:property name="contact_sensor_1_link" value="0.000001" />
   <!-- Property Blocks -->
   <xacro:property name="body_inertia">

File: rotors_description/urdf/hummingbird_base.xacro (robot description, xacro)
@@ -39,4 +39,8 @@
       wait_to_record_bag="$(arg wait_to_record_bag)" />
   </xacro:if>
+  <gazebo reference="${namespace}/base_link">
+    <mu1>0.99</mu1>
+    <mu2>0.99</mu2>
+  </gazebo>
   <!--<xacro:camera_macro
     namespace="${namespace}"
@@ -56,3 +60,34 @@
     <origin xyz="0 0 -0.05" rpy="0 1.57 0" />
   </xacro:camera_macro>-->
+<!--Contact sensor 1 Laser
+<joint name="contact_sensor_1_joint" type="fixed">
+    <axis xyz="0 1 0" />
+    <origin xyz="0 0 -0.1" rpy="0 0 0"/>
+    <parent link="${namespace}/base_link"/>
+    <child link="contact_sensor_1_link"/>
+  </joint>
+  <link name="contact_sensor_1_link">
+    <collision name="contact_sensor_collision_1">
+      <origin xyz="0 0 0" rpy="0 0 0"/>
+      <geometry>
+    	<box size="0.1 0.1 0.001"/>
+      </geometry>
+    </collision>
+    <visual name="contact_sensor_visual_1">
+      <origin xyz="0 0 0" rpy="0 0 0"/>
+      <geometry>
+    	<box size="0.01 0.01 0.001"/>
+      </geometry>
+    </visual>
+  </link>
+  <gazebo reference="contact_sensor_1_link">
+          <sensor name="contact_sensor_1" type="contact">
+		<plugin name="my_contact_plugin_1" filename="libgazebo_ros_bumper.so">
+			    <frameName>world</frameName>
+		</plugin>
+          <contact>
+            <collision>contact_sensor_collision_1_collision</collision>
+          </contact>
+      </sensor>
+  </gazebo>-->
 </robot>
