Commit message: Added files and worlds for RL laser-based navigation

File: rotors_description/urdf/component_snippets.xacro (robot description, xacro)
@@ -30,4 +30,58 @@
 	<waitToRecordBag>${wait_to_record_bag}</waitToRecordBag>
       </plugin>
+    </gazebo>
+  </xacro:macro>
+<!-- Macro to add Hokuyo range sensor -->
+<xacro:macro name="hokuyo_lidar" params="namespace parent_link">
+    <link name="${namespace}/hokuyo_link">
+      <inertial>
+         <mass value="0.01" />
+         <inertia ixx="1e-6" ixy="0.0" ixz="0.0" iyy="1e-6" iyz="0.0" izz="1e-6" />
+      </inertial>
+      <visual name="visual">
+        <geometry>
+          <mesh filename="package://rotors_description/meshes/hokuyo.dae" />
+        </geometry>
+      </visual>
+     </link>
+     <joint name="laser" type="fixed">
+      <parent link="${parent_link}" />
+      <child link="${namespace}/hokuyo_link" />
+      <origin xyz="0 0 0.05" rpy="0 0 0" />
+    </joint>
+    <gazebo reference="${namespace}/hokuyo_link">
+    <sensor type="gpu_ray" name="head_hokuyo_sensor">
+      <pose>0 0 0 0 0 0</pose>
+      <visualize>false</visualize>
+      <update_rate>40</update_rate>
+      <ray>
+        <scan>
+          <horizontal>
+            <samples>720</samples>
+            <resolution>1</resolution>
+            <min_angle>-2.35619</min_angle>
+            <max_angle>2.35619</max_angle>
+          </horizontal>
+        </scan>
+        <range>
+          <min>0.10</min>
+          <max>30.0</max>
+          <resolution>0.01</resolution>
+        </range>
+        <noise>
+          <type>gaussian</type>
+          <!-- Noise parameters based on published spec for Hokuyo laser
+               achieving "+-30mm" accuracy at range < 10m.  A mean of 0.0m and
+               stddev of 0.01m will put 99.7% of samples within 0.03m of the true
+               reading. -->
+          <mean>0.0</mean>
+          <stddev>0.01</stddev>
+        </noise>
+      </ray>
+      <plugin name="gazebo_ros_head_hokuyo_controller" filename="libgazebo_ros_gpu_laser.so">
+        <topicName>/drone11/scan</topicName>
+        <frameName>hokuyo_link</frameName>
+      </plugin>
+    </sensor>
     </gazebo>
   </xacro:macro>

File: rotors_description/urdf/hummingbird_laser.xacro (robot description, xacro)
@@ -60,38 +60,7 @@
     <origin xyz="0 0 -0.05" rpy="0 1.57 0" />
   </xacro:camera_macro>
-  <!-- <xacro:hokuyo_lidar
+  <xacro:hokuyo_lidar
     namespace="${namespace}"
-    parent_link="${namespace}/base_link" >
-  </xacro:hokuyo_lidar> -->
-<!--Contact sensor 1 Laser
-<joint name="contact_sensor_1_joint" type="fixed">
-    <axis xyz="0 1 0" />
-    <origin xyz="0 0 -0.1" rpy="0 0 0"/>
-    <parent link="${namespace}/base_link"/>
-    <child link="contact_sensor_1_link"/>
-  </joint>
-  <link name="contact_sensor_1_link">
-    <collision name="contact_sensor_collision_1">
-      <origin xyz="0 0 0" rpy="0 0 0"/>
-      <geometry>
-    	<box size="0.1 0.1 0.001"/>
-      </geometry>
-    </collision>
-    <visual name="contact_sensor_visual_1">
-      <origin xyz="0 0 0" rpy="0 0 0"/>
-      <geometry>
-    	<box size="0.01 0.01 0.001"/>
-      </geometry>
-    </visual>
-  </link>
-  <gazebo reference="contact_sensor_1_link">
-          <sensor name="contact_sensor_1" type="contact">
-		<plugin name="my_contact_plugin_1" filename="libgazebo_ros_bumper.so">
-			    <frameName>world</frameName>
-		</plugin>
-          <contact>
-            <collision>contact_sensor_collision_1_collision</collision>
-          </contact>
-      </sensor>
-  </gazebo>-->
+    parent_link="${namespace}/base_link" />
+  </xacro:hokuyo_lidar>
 </robot>
