Commit message: Added environments for test experiments in IROS 2018

File: rotors_description/urdf/firefly.xacro (robot description, xacro)
@@ -59,4 +59,18 @@
     <xacro:insert_block name="body_inertia" />
   </xacro:multirotor_base_macro>
+<!-- <xacro:cylinder_plugin_macro
+      namespace="${namespace}"
+      parent_link="${namespace}/base_link"
+      color="Red"
+      length_cylinder = "0.02"
+      radius_cylinder = "0.2">
+      <inertia ixx="0.00001" ixy="0.0" ixz="0.0" iyy="0.00001" iyz="0.0" izz="0.00001" />
+      <origin xyz="0 0 0.11" rpy="0 0 0" />
+    </xacro:cylinder_plugin_macro> ->
+<!--
+<xacro:bumper_plugin_macro
+      namespace="${namespace}"
+      parent_link="${namespace}/base_link">
+    </xacro:bumper_plugin_macro>-->
   <!-- Instantiate rotors -->
   <xacro:vertical_rotor
@@ -75,5 +89,5 @@
     rotor_drag_coefficient="${rotor_drag_coefficient}"
     rolling_moment_coefficient="${rolling_moment_coefficient}"
-    color="Red"
+    color="Green"
     use_own_mesh="false"
     mesh="">
@@ -178,5 +192,5 @@
     rotor_drag_coefficient="${rotor_drag_coefficient}"
     rolling_moment_coefficient="${rolling_moment_coefficient}"
-    color="Red"
+    color="Green"
     use_own_mesh="false"
     mesh="">

File: rotors_description/urdf/multirotor_base.xacro (robot description, xacro)
@@ -73,4 +73,47 @@
     </gazebo>
   </xacro:macro>
+  <!-- Macro to add an cylinder. -->
+  <xacro:macro name="cylinder_plugin_macro"
+    params="namespace parent_link color length_cylinder radius_cylinder *inertia *origin">
+    <!-- Cylinder link -->
+    <link name="${namespace}/cylinder_link">
+	<inertial>
+        <xacro:insert_block name="inertia" />
+        <mass value="0.001" />  <!-- [kg] -->
+        <origin xyz="0 0 0" rpy="0 0 0" />
+      </inertial>
+      <visual>
+          <origin xyz="0 0 0" rpy="0 0 0" />
+<geometry>
+	  <cylinder length="${length_cylinder}" radius="${radius_cylinder}" /> <!-- [m] -->
+</geometry>
+      </visual>
+    </link>
+	<gazebo reference="${namespace}/cylinder_link">
+      <material>Gazebo/${color}</material>
+    </gazebo>
+    <!-- Cylinder joint -->
+    <joint name="${namespace}/cylinder_joint" type="fixed">
+      <xacro:insert_block name="origin" />
+      <parent link="${parent_link}" />
+      <child link="${namespace}/cylinder_link" />
+      <limit upper="0" lower="0" effort="0" velocity="0" />
+    </joint>
+  </xacro:macro>
+  <!-- Macro to add bumper sensor. -->
+  <xacro:macro name="bumper_plugin_macro"
+    params="namespace parent_link">
+    <gazebo reference="${namespace}/base_link">
+	<sensor name="main_bumper" type="contact">
+    	<contact>
+       		<collision>${namespace}//base_link_inertia_collision</collision>
+    	</contact>
+    	<plugin name="gazebo_ros_bumper_controller" filename="libgazebo_ros_bumper.so">
+        	<bumperTopicName>bumper</bumperTopicName>
+        	<frameName>world</frameName>
+    	</plugin>
+	</sensor>
+    </gazebo>
+  </xacro:macro>
   <!-- Rotor joint and link -->
   <xacro:macro name="vertical_rotor"
