Commit message: added camera to hummingbird and some other models

File: rotors_description/urdf/hummingbird_base.xacro (robot description, xacro)
@@ -39,3 +39,20 @@
       wait_to_record_bag="$(arg wait_to_record_bag)" />
   </xacro:if>
+  <!--<xacro:camera_macro
+    namespace="${namespace}"
+    parent_link="${namespace}/base_link"
+    camera_suffix="bottom"
+    frame_rate="30"
+    horizontal_fov="2"
+    image_width="752"
+    image_height="480"
+    image_format="RGB8"
+    min_distance="0.02"
+    max_distance="50"
+    noise_mean="0.0"
+    noise_stddev="0.007"
+    enable_visual="true">
+    <box size="0.002 0.005 0.005" />
+    <origin xyz="0 0 -0.05" rpy="0 1.57 0" />
+  </xacro:camera_macro>-->
 </robot>

Commit message: adr iros race models and worlds

File: rotors_description/urdf/hummingbird_base.xacro (robot description, xacro)
@@ -46,8 +46,8 @@
     namespace="${namespace}"
     parent_link="${namespace}/base_link"
-    camera_suffix="bottom"
-    frame_rate="50"
-    horizontal_fov="2.3"
-    image_width="640"
+    camera_suffix="front"
+    frame_rate="30"
+    horizontal_fov="1.3463"
+    image_width="856"
     image_height="480"
     image_format="R8G8B8"
@@ -58,5 +58,5 @@
     enable_visual="true">
     <box size="0.002 0.005 0.005" />
-    <origin xyz="0 0 -0.05" rpy="0 1.57 0" />
+    <origin xyz="0.25 0 -0.05" rpy="0 0 0" />
   </xacro:camera_macro>
   <!-- <xacro:hokuyo_lidar
