Commit message: add the entire adr 2018 world to gazebo9

File: rotors_description/urdf/hummingbird_adr_base.xacro (robot description, xacro)
@@ -44,20 +44,20 @@
   </gazebo>
   <xacro:camera_macro
-    namespace="${namespace}"
-    parent_link="${namespace}/base_link"
-    camera_suffix="bottom"
-    frame_rate="50"
-    horizontal_fov="2.3"
-    image_width="640"
-    image_height="480"
-    image_format="R8G8B8"
-    min_distance="0.02"
-    max_distance="50"
-    noise_mean="0.0"
-    noise_stddev="0.007"
-    enable_visual="true">
-    <box size="0.002 0.005 0.005" />
-    <origin xyz="0 0 -0.05" rpy="0 1.57 0" />
-  </xacro:camera_macro>
+   namespace="${namespace}"
+   parent_link="${namespace}/base_link"
+   camera_suffix="front"
+   frame_rate="30"
+   horizontal_fov="1.3463"
+   image_width="856"
+   image_height="480"
+   image_format="R8G8B8"
+   min_distance="0.02"
+   max_distance="50"
+   noise_mean="0.0"
+   noise_stddev="0.007"
+   enable_visual="true">
+   <box size="0.002 0.005 0.005" />
+   <origin xyz="0.25 0 -0.05" rpy="0 0 0" />
+ </xacro:camera_macro>
   <!-- <xacro:hokuyo_lidar
     namespace="${namespace}"
